File: Front/FDU_V1/FDU_V1.kicad_sch (KiCad schematic)
At the start: 182 parts, among them IC1 SN65HVD230, IC10 XL1509-5.0E1, IC11 TDA2822D, IC12 AMS1117-3.3, IC3 74LVC3G17DC,125, IC4 STM32F103RBT6, IC5 MCP6291T-E_OT, IC6 LM2901, IC7 CD74HC30M96, IC8 74LVC3G17DC,125, IC9 SN74LVC3G04DCUR, J1 SWPROG, J2 WiFi serial interface, X1 S3D4.000000B20F30T, Y1 8MHz

Commit message: Changed microcontroller to 100pin
Parts:
- removed C11: 0.1uF, Capacitor_SMD:C_0805_2012Metric, symbol Device:C_Small
- removed IC4: STM32F103RBT6, Package_QFP:LQFP-64_10x10mm_P0.5mm, symbol MCU_ST_STM32F1:STM32F103RBTx
- removed X1: S3D4.000000B20F30T, Oscillator:Oscillator_SMD_EuroQuartz_XO32-4Pin_3.2x2.5mm, symbol Damo:S3D4.000000B20F30T
- added C11: 1uF 25V, Capacitor_SMD:CP_Elec_10x10, symbol Device:C_Polarized
- added C67, C68: 0.1uF, Capacitor_SMD:C_0805_2012Metric, symbol Device:C_Small
- added D14: SMAJ5.0A, Samacsys:DIOM5127X229N, symbol Samacsys:SMAJ5.0A
- added D16: SMAJ18CA, Samacsys:DIONM5127X229N, symbol Samacsys:SMAJ18CA
- added Q1, Q2: MMBT3904, Package_TO_SOT_SMD:SOT-23, symbol Transistor_BJT:MMBT3904
- added R68: 27K, Resistor_SMD:R_0805_2012Metric, symbol Device:R_Small
- added R69: 1K5, Resistor_SMD:R_0805_2012Metric, symbol Device:R_Small
- added R70: 4K7, Resistor_SMD:R_0805_2012Metric, symbol Device:R_Small
- added U1: STM32F103VCTx, Package_QFP:LQFP-100_14x14mm_P0.5mm, symbol MCU_ST_STM32F1:STM32F103VCTx
- R50, R58: value 1K2 -> 10K
- R52: value 2K2 -> 1K2
- R60: value 1K2 -> 100K
- R61: value 2K2 -> 100K
Connections:
- net +12V: now also R68.1
- net +3V3: now also C67.1, D14.1, U1.100 (VDD), U1.11 (VDD), U1.28 (VDD), U1.50 (VDD), U1.6 (VBAT), U1.75 (VDD); no longer R4.1
- net +5V: now also CONN6.16
- net BKIN: now also U1.51 (PB12)
- net BMS_IN: now also R12.1, U1.65 (PC8); no longer R12.2
- net BRAKE_IN: now also U1.3 (PE4)
- net CANRX0: now also U1.70 (PA11)
- net CANTX0: now also U1.71 (PA12)
- net CRUISE_IN: now also U1.91 (PB5)
- net DESAT_IN: now also U1.64 (PC7), U1.66 (PC9)
- net ENC_A: now also U1.31 (PA6)
- net ENC_B: now also U1.32 (PA7)
- net EXC_OUT: now also U1.83 (PD2)
- net FWD_IN: now also U1.29 (PA4)
- net GND: now also R12.2, R4.1, C11.2, C67.2, C68.1, D14.2, D16.2, Q1.2 (E), Q2.2 (E), R69.1, U1.10 (VSS), U1.19 (VSSA), U1.20 (VREF-), U1.27 (VSS), U1.49 (VSS), U1.74 (VSS), U1.99 (VSS); no longer IC10.4 (ON/OFF), R12.1, R52.2, R61.2
- net IL1_IN: now also U1.30 (PA5)
- net IL2_IN: now also U1.35 (PB0)
- net LINK DISCH: now also U1.78 (PC10)
- net OCUR_NEG: now also U1.93 (PB7)
- net OCUR_POS: now also U1.95 (PB8)
- net PWM_1N: now also U1.52 (PB13)
- net PWM_1P: now also U1.40 (PE9)
- net PWM_2N: now also U1.53 (PB14)
- net PWM_2P: now also U1.68 (PA9)
- net PWM_3N: now also U1.54 (PB15)
- net PWM_3P: now also U1.69 (PA10)
- net REV_IN: now also U1.63 (PC6)
- net START_IN: now also U1.92 (PB6)
- net SWCLK: now also U1.76 (PA14)
- net SWDAT: now also U1.72 (PA13)
- net THROTTLE 1: now also CONN6.12; no longer CONN6.15
- net THROTTLE 1 IN: now also U1.16 (PC1)
- net THROTTLE 2: now also CONN6.11; no longer CONN6.16
- net THROTTLE 2 IN: now also U1.15 (PC0)
- net TMPHS_IN: now also U1.33 (PC4)
- net TMPM1_IN: now also R50.2, U1.17 (PC2); no longer R52.1
- net TMPM2_IN: now also R52.1, R58.2, U1.24 (PA1); no longer R60.1, R61.1
- net TMPWTR_IN: now also U1.23 (PA0)
- net UDC_IN: now also U1.18 (PC3)
- net USART_RX: now also U1.48 (PB11)
- net USART_TX: now also U1.47 (PB10)
- net at C15.2, Y1.1: now also U1.12 (OSC_IN)
- net at C16.2, Y1.2: now also U1.13 (OSC_OUT)
- net +3V3A: now reaches C1.1, L1.1
- net +3V3A: now also C68.2, U1.21 (VREF+), U1.22 (VDDA)
- net at R63.1, R64.2: now also U1.34 (PC5)
- net at R3.1: now also U1.26 (PA3)
- net at R7.1: now also U1.37 (PB2)
- net at D1.1 (K): now also U1.80 (PC12)
- net at R4.2: now also U1.94 (BOOT0)
- net at C12.2: now also U1.14 (NRST)
- net 8Mhz Clock: now reaches IC3.1 (1A)
- net 8Mhz Clock: now also U1.67 (PA8)
- net MOT_TMP1_1 renamed MOT_TMP1
- net MOT_TMP1: now also R51.2; no longer R50.2
- net MOT_TMP1_2 renamed MOT_TMP2
- net MOT_TMP2: now also R52.2; no longer R51.2
- removed net MOT_TMP2_1: CONN6.11, R58.2
- net MOT_TMP2_2 renamed T15_OUT
- net T15_OUT: now also C11.1, R69.2, R70.2, U1.25 (PA2); no longer CONN6.12
- new net: Q2.1 (B), R61.1
- new net: IC10.4 (ON/OFF), Q1.3 (C), Q2.3 (C), R68.2
- new net: Q1.1 (B), R60.1
- new net MAIN_PSU_EN: R61.2, U1.77 (PA15)
- new net T15_IN: CONN6.15, D16.1, R70.1
Other:
- moved on the sheet: C1, C10, C12, C13, C14, C15, C16, C17, C18, C19, C2, C23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
